File: pcb/REV10/bpu-current_limiter.kicad_sch (KiCad schematic)
At the start: 45 parts, among them Q401 BCM857, Q402 SI2301, Q601 MMDT3906, Q602 SI2301, U403 AP2127, U601 LMV321A, U602 LMV331, U603 LMV321

Commit message: schematic cleanup
Other:
- note removed: "Additional Filter PWM from MCU"
Changed lines of the file:
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@@
-    (stroke (width 0) (type default))
-  )
-  (polyline (pts (xy 107.95 68.58) (xy 72.39 68.58))
     (stroke (width 0) (type default))
   )
@@
     (stroke (width 0) (type default))
   )
-  (polyline (pts (xy 72.39 53.34) (xy 107.95 53.34))
-    (stroke (width 0) (type default))
-  )
   (wire (pts (xy 146.05 130.81) (xy 146.05 128.27))
     (stroke (width 0) (type default))
@@
     (stroke (width 0) (type default))
   )
-  (polyline (pts (xy 72.39 68.58) (xy 72.39 53.34))
-    (stroke (width 0) (type default))
-  )
   (wire (pts (xy 149.86 46.99) (xy 143.51 46.99))
     (stroke (width 0) (type default))
@@
   )
   (wire (pts (xy 40.64 45.72) (xy 31.75 45.72))
-    (stroke (width 0) (type default))
-  )
-  (polyline (pts (xy 107.95 53.34) (xy 107.95 68.58))
     (stroke (width 0) (type default))
   )
@@
     (effects (font (size 1.27 1.27)) (justify left bottom))
   )
-  (text "Additional Filter\nPWM from MCU" (at 76.2 64.77 0)
-    (effects (font (size 1.27 1.27)) (justify left bottom))
-  )
