File: pcb/7-REV0/micro-rp2040.kicad_sch (KiCad schematic)
At the start: 50 parts, among them J201 Conn_01x03, J202 TYPE-C-31-M-12, SW101 TS3425BA 098 2.5H 250gf, SW102 TS3315A 250gf 025, U1 RP2350B, U102 W25Q128JVSIQ, U105 MT29F1G01ABAFDWB, U3 TLV74311PDBVR, U401 ME6211A33PG-N, U8 APS6404L-3SQR-ZR, Y101 ABM8-272-T3

Commit message: minor updates to collaborative board redesign
Parts:
- removed R101: 1K, Resistor_SMD:R_0402_1005Metric, symbol Device:R_Small
- added C21: 10uF, Capacitor_SMD:C_0402_1005Metric, symbol Device:C_Small
- added C22: 0.1uF, Capacitor_SMD:C_0402_1005Metric, symbol Device:C_Small
- added Q1, Q2: MMBT7002K, Package_TO_SOT_SMD:SOT-23, symbol Transistor_FET:BSS138
- added R10: 470K, Resistor_SMD:R_0402_1005Metric, symbol Device:R_Small
- added R11, R8, R9: 10K, Resistor_SMD:R_0402_1005Metric, symbol Device:R_Small
- added R12: 1K, Resistor_SMD:R_0402_1005Metric, symbol Device:R_Small
Connections:
- net +3V3: now also SW101.1 (A), R8.1, R9.1; no longer U1.35 (RUN)
- net AMUX_OUT: now also U1.56 (GPIO45_ADC5); no longer U1.57 (GPIO46_ADC6)
- net BUTTONS: now also U1.55 (GPIO44_ADC4); no longer U1.54 (GPIO43_ADC3)
- net CURRENT_SENSE: now also U1.57 (GPIO46_ADC6); no longer U1.58 (GPIO47_ADC7)
- net DISPLAY_RESET: now also U1.45 (GPIO36); no longer U1.38 (GPIO30)
- net GND: now also C21.2, C22.2, Q1.2 (S), Q2.2 (S), R11.2; no longer SW101.2 (B)
- net QSPI_SS_2: now also U1.58 (GPIO47_ADC7)
- net RGB_CDO: now also U1.38 (GPIO30); no longer U1.45 (GPIO36)
- net I2C_RESET: now reaches U1.46 (GPIO37)
- net I2C_SDA: now reaches U1.53 (GPIO42_ADC2)
- net I2C_SDA: now also R8.2
- net QSPI_SS renamed MCU_BOOTLOAD
- net MCU_BOOTLOAD: now also R12.2
- new net: C21.1, Q2.1 (G), R10.2
- new net: Q1.1 (G), R10.1, R11.1
- new net: Q2.3 (D), R12.1
- new net I2C_SCL: R9.2, U1.54 (GPIO43_ADC3)
- new net MCU_RESET: C22.1, Q1.3 (D), U1.35 (RUN)
Other:
- note added: "AMUX_OUT, CURRENT_SENSE moved 1 pin"
- note added: "BUTTONS moved 1 pin"
- note added: "Pin for I2C RESET (100K pull-up)"
- note added: "Relocated for RGB_CDO"
- note removed: "DISPLAY_ pins and FLASH_CS can be swapped for easiest routing"
- note removed: "GPIO44/45 are SDA0/SCL0"
- note removed: "Pin for I2C RESET?"
- note removed: "The 4 CURRENT_ pins can be swapped for easiest routing"
- moved on the sheet: SW101
