File: pcb/7-REV0/pull-x-resistors.kicad_sch (KiCad schematic)
At the start: 14 parts, among them U6 TCA6416RTWT, U7 TCA6416RTWT

Commit message: remove old pullups, remove 1M pull-down. Add footprints and updated PCB.
Parts:
- U6, U7: footprint TCA6416RTWT:QFN50P400X400X80-25N -> qfn24-4x4x50:QFN50P400X400X80-25N
Changed lines of the file:
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@@
 			)
 		)
-		(property "Footprint" "TCA6416RTWT:QFN50P400X400X80-25N"
+		(property "Footprint" "qfn24-4x4x50:QFN50P400X400X80-25N"
 			(at 87.63 92.71 0)
 			(effects
@@
 			)
 		)
-		(property "Footprint" "TCA6416RTWT:QFN50P400X400X80-25N"
+		(property "Footprint" "qfn24-4x4x50:QFN50P400X400X80-25N"
 			(at 167.64 92.71 0)
 			(effects

Commit message: minor updates to collaborative board redesign
Parts:
- added R7: 100K, Resistor_SMD:R_0402_1005Metric, symbol Device:R_Small
Connections:
- net +3V3: now also R7.1
- net I2C_RESET: now also R7.2
Changed lines of the file:
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@@
 	)
 	(junction
+		(at 67.31 74.93)
+		(diameter 0)
+		(color 0 0 0 0)
+	)
+	(junction
 		(at 109.22 69.85)
 		(diameter 0)
@@
 	(wire
 		(pts
+			(xy 67.31 74.93) (xy 69.85 74.93)
+		)
+		(stroke
+			(width 0)
+			(type default)
+		)
+	)
+	(wire
+		(pts
 			(xy 64.77 92.71) (xy 59.69 92.71)
 		)
@@
 	(wire
 		(pts
+			(xy 60.96 74.93) (xy 67.31 74.93)
+		)
+		(stroke
+			(width 0)
+			(type default)
+		)
+	)
+	(wire
+		(pts
 			(xy 64.77 95.25) (xy 59.69 95.25)
 		)
@@
 	(global_label "I2C_RESET"
 		(shape input)
-		(at 69.85 74.93 180)
+		(at 60.96 74.93 180)
 		(fields_autoplaced yes)
 		(effects
@@
 		)
 		(property "Intersheetrefs" "${INTERSHEET_REFS}"
-			(at 57.722 74.93 0)
+			(at 48.832 74.93 0)
 			(effects
 				(font
@@
 	)
 	(symbol
+		(lib_id "Device:R_Small")
+		(at 67.31 72.39 0)
+		(unit 1)
+		(exclude_from_sim no)
+		(in_bom yes)
+		(on_board yes)
+		(dnp no)
+		(property "Reference" "R7"
+			(at 66.04 71.12 0)
+			(effects
+				(font
+					(size 1.27 1.27)
+				)
+				(justify right)
+			)
+		)
+		(property "Value" "100K"
+			(at 66.04 73.66 0)
+			(effects
+				(font
+					(size 1.27 1.27)
+				)
+				(justify right)
+			)
+		)
+		(property "Footprint" "Resistor_SMD:R_0402_1005Metric"
+			(at 67.31 72.39 0)
+			(effects
+				(font
+					(size 1.27 1.27)
+				)
+				(hide yes)
+			)
+		)
+		(property "Datasheet" "~"
+			(at 67.31 72.39 0)
+			(effects
+				(font
+					(size 1.27 1.27)
+				)
+				(hide yes)
+			)
+		)
+		(property "Description" ""
+			(at 67.31 72.39 0)
+			(effects
+				(font
+					(size 1.27 1.27)
+				)
+				(hide yes)
+			)
+		)
+		(property "RMB" "0.005749"
+			(at 67.31 72.39 0)
+			(effects
+				(font
+					(size 1.27 1.27)
+				)
+				(hide yes)
+			)
+		)
+		(property "Supplier" "https://item.szlcsc.com/61543.html"
+			(at 67.31 72.39 0)
+			(effects
+				(font
+					(size 1.27 1.27)
+				)
+				(hide yes)
+			)
+		)
+		(pin "1"
+		)
+		(pin "2"
+		)
+		(instances
+			(project "7-REV0"
+				(path "/1f56410a-eaac-4444-b0f7-cfd3531e22ac/70d89944-cef2-4c07-9520-6c47f8613415"
+					(reference "R7")
+					(unit 1)
+				)
+			)
+		)
+	)
+	(symbol
 		(lib_id "dp-rarray:R_Array")
 		(at 107.95 102.87 270)
@@
 				)
 			)
+		)
+	)
+	(symbol
+		(lib_id "BusPirate-5-rev10-rescue:+3.3V-power")
+		(at 67.31 69.85 0)
+		(unit 1)
+		(exclude_from_sim no)
+		(in_bom yes)
+		(on_board yes)
+		(dnp no)
+		(property "Reference" "#PWR06"
+			(at 67.31 73.66 0)
+			(effects
+				(font
+					(size 1.27 1.27)
+				)
+				(hide yes)
+			)
+		)
+		(property "Value" "+3V3"
+			(at 67.691 65.4558 0)
+			(effects
+				(font
+					(size 1.27 1.27)
+				)
+			)
+		)
+		(property "Footprint" ""
+			(at 67.31 69.85 0)
+			(effects
+				(font
+					(size 1.27 1.27)
+				)
+				(hide yes)
+			)
+		)
+		(property "Datasheet" ""
+			(at 67.31 69.85 0)
+			(effects
+				(font
+					(size 1.27 1.27)
+				)
+				(hide yes)
+			)
+		)
+		(property "Description" ""
+			(at 67.31 69.85 0)
+			(effects
+				(font
+					(size 1.27 1.27)
+				)
+				(hide yes)
+			)
+		)
+		(pin "1"
+		)
+		(instances
+			(project "7-REV0"
+				(path "/1f56410a-eaac-4444-b0f7-cfd3531e22ac/70d89944-cef2-4c07-9520-6c47f8613415"
+					(reference "#PWR06")
+					(unit 1)
+				)
+			)
