File: pcb/7-REVA-PC1/7-REVA-PC1.kicad_pcb (KiCad board)
At the start: 4 copper layers, 60 x 60 mm, 260 parts, among them J201 Conn_01x03, J202 TYPE-C-31-M-12, J301 Conn_01x10, J302 Conn_01x09, Q1 MMBT7002K, Q2 MMBT7002K, Q202 MMBT7002K, Q401 BCM857, Q402 BC2301T 2.8A, Q601 MMDT3906, Q602 BC2301T 2.8A, SW101 TS3425BA 098 2.5H 250gf, SW102 TS3315A 250gf 025, U1 RP2350B, U10 LM358_DFN, U102 W25Q128JVSIQ, U105 MT29F1G01ABAFDWB, U11 LM358_DFN, U12 LM358_DFN, U13 LM358_DFN, U14 IP4220CZ6F, U15 IP4220CZ6F, U2 74LVC8T245BQ, U3 TLV74311PDBVR, U301 AiP74LVC1T45GC363.TR, U302 AiP74LVC1T45GC363.TR, U303 AiP74LVC1T45GC363.TR, U304 AiP74LVC1T45GC363.TR, U305 AiP74LVC1T45GC363.TR, U306 AiP74LVC1T45GC363.TR, U307 AiP74LVC1T45GC363.TR, U308 AiP74LVC1T45GC363.TR, U4 MCP4725xxx-xCH, U401 ME6211A33PG-N, U402 CD4067, U403 AP2127, U5 MCP4725xxx-xCH, U503 74HCT245BQ, U6 TCA6416RTWT, U601 GS321A-TR, U602 GSV331-TR, U7 TCA6416RTWT, U8 APS6404L-3SQR-ZR, U9 LM358_DFN, Y101 ABM8-272-T3

Commit message: 7R1 PCB routed
Parts:
- removed C103, C12, C121: 0.1uF, Capacitor_SMD:C_0402_1005Metric
- removed C13, C6: 10uF, Capacitor_SMD:C_0805_2012Metric
- removed C21: 10uF, Capacitor_SMD:C_0402_1005Metric
- removed C603: DNF, Capacitor_SMD:C_0402_1005Metric
- removed D11, D12, D13, D14, D15, D16, D17, D18: DESD5Z5.0, Diode_SMD:D_SOD-523
- removed D601: 1N4148WT, Diode_SMD:D_SOD-523
- removed Q202: MMBT7002K, Package_TO_SOT_SMD:SOT-23
- removed R102: DNF, Resistor_SMD:R_0402_1005Metric
- removed R208, R612: 200R, Resistor_SMD:R_0402_1005Metric
- removed R3, R320, R5: 510R, Resistor_SMD:R_0402_1005Metric
- removed R7: 100K, Resistor_SMD:R_0402_1005Metric
- removed RN315, RN400, RN401: 510R, Resistor_SMD:R_Array_Convex_4x0402
- added C23: 10uF/6.3v, Capacitor_SMD:C_0402_1005Metric, F.Cu at (137.0, 106.5)
- added C24: 10uF/6.3v, Capacitor_SMD:C_0402_1005Metric, F.Cu at (134.0, 74.6)
- added C29: 10uF/6.3v, Capacitor_SMD:C_0402_1005Metric, F.Cu at (125.2, 106.5)
- added C36: 10uF/6.3v, Capacitor_SMD:C_0402_1005Metric, F.Cu at (147.8, 74.5)
- added C413: 10uF/6.3V, Capacitor_SMD:C_0402_1005Metric, F.Cu at (115.2, 82.2)
- added C415: 0.1uF, Capacitor_SMD:C_0402_1005Metric, F.Cu at (140.2, 87.0)
- added C416: 0.1uF, Capacitor_SMD:C_0402_1005Metric, F.Cu at (140.2, 85.0)
- added Q5: 2N7002KT, library:SOT-523, F.Cu at (153.5, 74.5)
- added R414: 10K, Resistor_SMD:R_0402_1005Metric, F.Cu at (138.5, 86.0)
- added R415: 10K, Resistor_SMD:R_0402_1005Metric, F.Cu at (138.5, 85.0)
- added RN10: 1M, Resistor_SMD:R_Array_Convex_4x0402, F.Cu at (130.2, 99.8)
- added RN11: 1M, Resistor_SMD:R_Array_Convex_4x0402, F.Cu at (133.2, 99.8)
- added U16: SP3002-04JTG, Package_TO_SOT_SMD:SOT-363_SC-70-6, F.Cu at (132.8, 71.5)
- C10, C11, C201, C202, C401, C402, C404, C407: value 4.7uF -> 10uF/6.3v
- C104, C109, C19, C4, C601: value 2.2uF -> 10uF/6.3v
- C18: value 0.1uF -> 10uF/6.3v
- D1, D2, D3, D4, D5, D6, D7, D8, D9, Q402, Q602: footprint Package_TO_SOT_SMD:SOT-523 -> library:SOT-523
- D10: value DESD5Z5.0 -> SMF5.0A; footprint Diode_SMD:D_SOD-523 -> Diode_SMD:D_SMF
- Q1, Q2: value MMBT7002K -> 2N7002KT; footprint Package_TO_SOT_SMD:SOT-23 -> library:SOT-523
- R13, R14, R15, R16, R17, R18, R19, R20: value 120R -> 120R 0.5W; footprint Resistor_SMD:R_0805_2012Metric -> Resistor_SMD:R_0805_2012Metric_Pad1.20x1.40mm_HandSolder
- R202, R203: value 22R -> 27R
- R6: value 100K -> 10K
- RN301, RN306: value 330R -> 120R
- RN302, RN307: value 100K -> 4.7K
- U14, U15: value IP4220CZ6F -> SP3002-04JTG; footprint library:SOT95P275X110-6N -> Package_TO_SOT_SMD:SOT-363_SC-70-6
- U4: value MCP4725xxx-xCH -> XL9555QF24; footprint Package_TO_SOT_SMD:SOT-23-6 -> Package_DFN_QFN:QFN-24-1EP_4x4mm_P0.5mm_EP2.7x2.7mm
- U403: value AP2127 -> AP2127K-ADJ
- U5: value MCP4725xxx-xCH -> LM358_DFN; footprint Package_TO_SOT_SMD:SOT-23-6 -> Package_DFN_QFN:DFN-8-1EP_2x2mm_P0.5mm_EP1.05x1.75mm
- U6, U7: value TCA6416RTWT -> TCA6416ARTWR; footprint qfn24-4x4x50:QFN50P400X400X80-25N -> Package_DFN_QFN:QFN-24-1EP_4x4mm_P0.5mm_EP2.75x2.75mm
- U8: footprint Package_SON:Winbond_USON-8-1EP_3x2mm_P0.5mm_EP0.2x1.6mm -> library:USON-8-3x2mm_P0.5mm_EPthin
- moved R20 58.0 mm to (141.8, 108.8), turned to -90 degrees
- moved R19 55.4 mm to (139.5, 108.8), turned to -90 degrees
- moved R18 50.2 mm to (134.5, 108.8), turned to -90 degrees
- moved R17 47.9 mm to (132.2, 108.8), turned to -90 degrees
- moved U15 47.8 mm to (137.0, 108.8), turned to 90 degrees
- moved R16 45.8 mm to (130.0, 108.8), turned to -90 degrees
- moved R15 43.9 mm to (127.8, 108.8), turned to -90 degrees
- moved R8 40.2 mm to (106.0, 109.2), turned to 0 degrees
- moved R9 40.0 mm to (106.0, 108.0), turned to 0 degrees
- moved R14 39.6 mm to (122.8, 108.8), turned to -90 degrees
- moved R13 38.3 mm to (120.5, 108.8), turned to -90 degrees
- moved U14 34.5 mm to (125.2, 108.8), turned to 90 degrees
- moved C18 20.7 mm to (142.8, 84.5), turned to 0 degrees
- moved Q2 20.0 mm to (141.2, 95.8), turned to 180 degrees
- moved C510 19.8 mm to (152.0, 100.5), turned to 90 degrees
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Connections:
- net BPIO1 renamed BPIO1_TVS
- net BPIO2 renamed BPIO2_TVS
- net BPIO3 renamed BPIO3_TVS
- net BPIO4 renamed BPIO4_TVS
- net BPIO5 renamed BPIO5_TVS
- net BPIO6 renamed BPIO6_TVS
- net BPIO7 renamed BPIO7_TVS
- net LA_BPIO0 renamed LA_BPIO0_TVS
- net LA_BPIO1 renamed LA_BPIO1_TVS
- net LA_BPIO2 renamed LA_BPIO2_TVS
- net LA_BPIO3 renamed LA_BPIO3_TVS
- net LA_BPIO4 renamed LA_BPIO4_TVS
- net LA_BPIO5 renamed LA_BPIO5_TVS
- net LA_BPIO6 renamed LA_BPIO6_TVS
- net LA_BPIO7 renamed LA_BPIO7_TVS
- C5 pad 1: +3V3 -> GND
- C5 pad 2: GND -> +3V3
- D10 pad 1: BPIO0 -> VREF_VOUT
- LCD201 pad 2: DISPLAY_LED-K -> Net-(LCD201-LED-K)
- LCD201 pad 3: +VUSB -> Net-(LCD201-LED-A)
- Q1 pad 3: MCU_RESET -> Net-(Q1-D)
- Q2 pad 1: Net-(Q2-G) -> DISPLAY_BACKLIGHT
- Q2 pad 3: Net-(Q2-D) -> Net-(LCD201-LED-K)
- Q602 pad 1: Net-(Q602-G) -> CURRENT_EN
- R10 pad 1: Net-(Q1-G) -> Net-(Q5-G)
- R10 pad 2: Net-(Q2-G) -> Net-(Q1-G)
- R11 pad 1: Net-(Q1-G) -> Net-(Q5-G)
- R12 pad 1: Net-(Q2-D) -> Net-(Q1-D)
- R13 pad 1: BPIO0 -> BPIO0_TVS
- R209 pad 1: Net-(Q202-D) -> +VUSB
- R209 pad 2: DISPLAY_LED-K -> Net-(LCD201-LED-A)
- RN318 pad 5: BPIO0 -> BPIO0_TVS
- RN6 pad 4: BPIO0 -> BPIO0_TVS
- RN7 pad 4: BPIO0 -> BPIO0_TVS
- RN8 pad 8: BPIO0 -> BPIO0_TVS
- RN9 pad 8: BPIO0 -> BPIO0_TVS
- SW101 pad 2: Net-(Q1-G) -> Net-(Q5-G)
- U1 pad 16: CURRENT_EN_OVERRIDE -> XL9555_~{INT}
- U1 pad 17: CURRENT_RESET -> unconnected-(U1-GPIO17-Pad17)
- U1 pad 18: CURRENT_EN -> I2C_SDA
- U1 pad 19: CURRENT_DETECT -> I2C_SCL
- U1 pad 42: DISPLAY_BACKLIGHT -> unconnected-(U1-GPIO33-Pad42)
- U1 pad 45: DISPLAY_RESET -> unconnected-(U1-GPIO36-Pad45)
- U1 pad 53: I2C_SDA -> VREG_ADJ_MCU
- U1 pad 54: I2C_SCL -> CURRENT_ADJ_MCU
- U10 pad 1: MUX_BPIO2 -> MUX_BPIO2_TVS
- U10 pad 2: MUX_BPIO2 -> MUX_BPIO2_TVS
- U10 pad 6: MUX_BPIO3 -> MUX_BPIO3_TVS
- U10 pad 7: MUX_BPIO3 -> MUX_BPIO3_TVS
- U11 pad 1: MUX_BPIO4 -> MUX_BPIO4_TVS
- U11 pad 2: MUX_BPIO4 -> MUX_BPIO4_TVS
- U11 pad 6: MUX_BPIO5 -> MUX_BPIO5_TVS
- U11 pad 7: MUX_BPIO5 -> MUX_BPIO5_TVS
- U12 pad 1: MUX_BPIO6 -> MUX_BPIO6_TVS
- U12 pad 2: MUX_BPIO6 -> MUX_BPIO6_TVS
- U12 pad 6: MUX_BPIO7 -> MUX_BPIO7_TVS
- U12 pad 7: MUX_BPIO7 -> MUX_BPIO7_TVS
- U14 pad 1: BPIO0 -> BPIO0_TVS
- U2 pad 14: BPIO0 -> BPIO0_TVS
- U301 pad 4: BPIO0 -> BPIO0_TVS
- U4 pad 1: CURRENT_ADJ_MCU -> Net-(RN10A-R1.8)
- U4 pad 2: GND -> Net-(RN10B-R1.8)
- U4 pad 3: +3V3 -> Net-(RN10C-R1.8)
- U4 pad 4: I2C_SDA -> Net-(RN10D-R1.8)
- U4 pad 5: I2C_SCL -> Net-(RN11A-R1.8)
- U4 pad 6: GND -> Net-(RN11B-R1.8)
- U402 pad 2: Net-(RN401D-R1.1) -> MUX_BPIO0_TVS
- U402 pad 21: Net-(U402-I10) -> VREG_OUT
- U402 pad 22: Net-(U402-I9) -> MUX_VREF_VOUT
- U402 pad 23: Net-(U402-I8) -> +VUSB
- U402 pad 3: Net-(RN401C-R1.1) -> MUX_BPIO1_TVS
- U402 pad 4: Net-(RN401B-R1.1) -> MUX_BPIO2_TVS
- U402 pad 5: Net-(RN401A-R1.1) -> MUX_BPIO3_TVS
- U402 pad 6: Net-(RN400D-R1.1) -> MUX_BPIO4_TVS
- U402 pad 7: Net-(RN400C-R1.1) -> MUX_BPIO5_TVS
- U402 pad 8: Net-(RN400B-R1.1) -> MUX_BPIO6_TVS
- U402 pad 9: Net-(RN400A-R1.1) -> MUX_BPIO7_TVS
- U5 pad 2: GND -> VREG_ADJ
- U5 pad 3: +3V3 -> Net-(U5A-+)
- U5 pad 4: I2C_SDA -> GND
- U5 pad 5: I2C_SCL -> Net-(U5B-+)
- U5 pad 6: +3V3 -> CURRENT_ADJ
- U503 pad 14: Net-(RN315A-R1.8) -> AMUX_S3
- U503 pad 15: Net-(RN315B-R1.8) -> AMUX_S2
- U503 pad 16: Net-(RN315C-R1.8) -> AMUX_S1
- U503 pad 17: Net-(RN315D-R1.8) -> AMUX_S0
- U6 pad 25: unconnected-(U6-EP-Pad25) -> GND
- U602 pad 1: CURRENT_ADJ_MCU -> CURRENT_ADJ
- U7 pad 25: unconnected-(U7-EP-Pad25) -> GND
- U9 pad 1: MUX_BPIO0 -> MUX_BPIO0_TVS
- U9 pad 2: MUX_BPIO0 -> MUX_BPIO0_TVS
- U9 pad 6: MUX_BPIO1 -> MUX_BPIO1_TVS
- U9 pad 7: MUX_BPIO1 -> MUX_BPIO1_TVS
Routing:
- net BPIO0: track 83.3 -> 0.00 mm, vias 4 -> 0
- net BPIO0_TVS: track 0.00 -> 72.4 mm, vias 0 -> 4
- net DISPLAY_BACKLIGHT: track 2.39 -> 43.7 mm, vias 0 -> 2
- net Net-(U5A-+): track 0.00 -> 35.7 mm, vias 0 -> 3
- net Net-(RN318A-R1.1): track 8.30 -> 43.8 mm
- net Net-(U5B-+): track 0.00 -> 35.4 mm, vias 0 -> 3
- net Net-(RN11D-R1.8): track 0.00 -> 35.2 mm, vias 0 -> 2
- net Net-(RN318B-R1.1): track 4.27 -> 38.2 mm, vias 0 -> 2
- net Net-(RN11C-R1.8): track 0.00 -> 32.9 mm, vias 0 -> 2
- net Net-(RN11B-R1.8): track 0.00 -> 30.7 mm, vias 0 -> 2
- net DISPLAY_RESET: track 4.44 -> 34.1 mm
- net Net-(RN11A-R1.8): track 0.00 -> 29.6 mm, vias 0 -> 2
- net Net-(RN10D-R1.8): track 0.00 -> 28.2 mm, vias 0 -> 2
- net Net-(RN10C-R1.8): track 0.00 -> 27.2 mm, vias 0 -> 2
- net Net-(RN318C-R1.1): track 5.98 -> 32.5 mm, vias 0 -> 2
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- added copper zone on B.Cu, net GND
- added copper zone on F.Cu, net Net-(LCD201-LED-K)
- removed copper zone on B.Cu, net VREG_OUT
Other:
- board text added: "7R1B"
- board text added: "MAR 2025"
- board text added: "REV 1B"
- board text removed: "NOV 2024"
- board text removed: "Nov 2024"
- board text removed: "REV 0A"
