File: pcb/7-REVA-PC1/bpu-iobufffer.kicad_sch (KiCad schematic)
At the start: 45 parts, among them J301 Conn_01x10, J302 Conn_01x09, U14 SP3002-04JTG, U15 SP3002-04JTG, U301 AiP74LVC1T45GC363.TR, U302 AiP74LVC1T45GC363.TR, U303 AiP74LVC1T45GC363.TR, U304 AiP74LVC1T45GC363.TR, U305 AiP74LVC1T45GC363.TR, U306 AiP74LVC1T45GC363.TR, U307 AiP74LVC1T45GC363.TR, U308 AiP74LVC1T45GC363.TR

Commit message: 7R1 PCB routed
Parts:
- RN301, RN306: value 330R -> 120R
- RN302, RN307: value 100K -> 4.7K
Changed lines of the file:
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@@
 		(dnp no)
 		(property "Reference" "RN301"
-			(at 33.02 33.02 90)
-			(effects
-				(font
-					(size 1.27 1.27)
-				)
-			)
-		)
-		(property "Value" "330R"
-			(at 33.02 37.9476 90)
+			(at 33.274 38.354 90)
+			(effects
+				(font
+					(size 1.27 1.27)
+				)
+			)
+		)
+		(property "Value" "120R"
+			(at 33.02 40.64 90)
 			(effects
 				(font
@@
 		(dnp no)
 		(property "Reference" "RN302"
-			(at 33.02 35.56 90)
-			(effects
-				(font
-					(size 1.27 1.27)
-				)
-			)
-		)
-		(property "Value" "100K"
-			(at 33.02 40.4876 90)
+			(at 33.02 45.466 90)
+			(effects
+				(font
+					(size 1.27 1.27)
+				)
+			)
+		)
+		(property "Value" "4.7K"
+			(at 33.02 43.18 90)
 			(effects
 				(font
@@
 		(dnp no)
 		(property "Reference" "RN301"
-			(at 34.29 88.9 90)
-			(effects
-				(font
-					(size 1.27 1.27)
-				)
-			)
-		)
-		(property "Value" "330R"
-			(at 34.29 93.8276 90)
+			(at 34.29 94.234 90)
+			(effects
+				(font
+					(size 1.27 1.27)
+				)
+			)
+		)
+		(property "Value" "120R"
+			(at 34.29 96.52 90)
 			(effects
 				(font
@@
 		(dnp no)
 		(property "Reference" "RN302"
-			(at 34.29 91.44 90)
-			(effects
-				(font
-					(size 1.27 1.27)
-				)
-			)
-		)
-		(property "Value" "100K"
-			(at 34.29 96.52 90)
+			(at 34.29 101.346 90)
+			(effects
+				(font
+					(size 1.27 1.27)
+				)
+			)
+		)
+		(property "Value" "4.7K"
+			(at 34.29 99.06 90)
 			(effects
 				(font
@@
 		(dnp no)
 		(property "Reference" "RN301"
-			(at 97.79 31.75 90)
-			(effects
-				(font
-					(size 1.27 1.27)
-				)
-			)
-		)
-		(property "Value" "330R"
-			(at 97.79 36.6776 90)
+			(at 97.79 36.83 90)
+			(effects
+				(font
+					(size 1.27 1.27)
+				)
+			)
+		)
+		(property "Value" "120R"
+			(at 97.79 39.37 90)
 			(effects
 				(font
@@
 		(dnp no)
 		(property "Reference" "RN302"
-			(at 97.79 34.29 90)
-			(effects
-				(font
-					(size 1.27 1.27)
-				)
-			)
-		)
-		(property "Value" "100K"
-			(at 97.79 39.37 90)
+			(at 97.79 43.942 90)
+			(effects
+				(font
+					(size 1.27 1.27)
+				)
+			)
+		)
+		(property "Value" "4.7K"
+			(at 97.79 41.91 90)
 			(effects
 				(font
@@
 		(dnp no)
 		(property "Reference" "RN301"
-			(at 97.79 87.63 90)
-			(effects
-				(font
-					(size 1.27 1.27)
-				)
-			)
-		)
-		(property "Value" "330R"
-			(at 97.79 92.5576 90)
+			(at 97.79 92.71 90)
+			(effects
+				(font
+					(size 1.27 1.27)
+				)
+			)
+		)
+		(property "Value" "120R"
+			(at 97.79 95.25 90)
 			(effects
 				(font
@@
 		(dnp no)
 		(property "Reference" "RN306"
-			(at 166.37 33.02 90)
-			(effects
-				(font
-					(size 1.27 1.27)
-				)
-			)
-		)
-		(property "Value" "330R"
-			(at 166.37 37.9476 90)
+			(at 166.37 38.1 90)
+			(effects
+				(font
+					(size 1.27 1.27)
+				)
+			)
+		)
+		(property "Value" "120R"
+			(at 166.37 40.64 90)
 			(effects
 				(font
@@
 		(dnp no)
 		(property "Reference" "RN302"
-			(at 97.79 90.17 90)
-			(effects
-				(font
-					(size 1.27 1.27)
-				)
-			)
-		)
-		(property "Value" "100K"
-			(at 97.79 95.25 90)
+			(at 97.79 100.076 90)
+			(effects
+				(font
+					(size 1.27 1.27)
+				)
+			)
+		)
+		(property "Value" "4.7K"
+			(at 97.79 97.79 90)
 			(effects
 				(font
@@
 		(dnp no)
 		(property "Reference" "RN307"
-			(at 166.37 35.56 90)
-			(effects
-				(font
-					(size 1.27 1.27)
-				)
-			)
-		)
-		(property "Value" "100K"
-			(at 166.37 40.64 90)
+			(at 166.37 45.212 90)
+			(effects
+				(font
+					(size 1.27 1.27)
+				)
+			)
+		)
+		(property "Value" "4.7K"
+			(at 166.37 43.18 90)
 			(effects
 				(font
@@
 		(dnp no)
 		(property "Reference" "RN306"
-			(at 233.68 83.82 90)
-			(effects
-				(font
-					(size 1.27 1.27)
-				)
-			)
-		)
-		(property "Value" "330R"
-			(at 233.68 88.7476 90)
+			(at 233.68 88.9 90)
+			(effects
+				(font
+					(size 1.27 1.27)
+				)
+			)
+		)
+		(property "Value" "120R"
+			(at 233.68 91.44 90)
 			(effects
 				(font
@@
 		(dnp no)
 		(property "Reference" "RN307"
-			(at 233.68 86.36 90)
-			(effects
-				(font
-					(size 1.27 1.27)
-				)
-			)
-		)
-		(property "Value" "100K"
-			(at 233.68 91.44 90)
+			(at 233.68 96.012 90)
+			(effects
+				(font
+					(size 1.27 1.27)
+				)
+			)
+		)
+		(property "Value" "4.7K"
+			(at 233.68 94.234 90)
 			(effects
 				(font
@@
 		(dnp no)
 		(property "Reference" "RN306"
-			(at 238.76 31.75 90)
-			(effects
-				(font
-					(size 1.27 1.27)
-				)
-			)
-		)
-		(property "Value" "330R"
-			(at 238.76 36.6776 90)
+			(at 238.76 36.83 90)
+			(effects
+				(font
+					(size 1.27 1.27)
+				)
+			)
+		)
+		(property "Value" "120R"
+			(at 238.76 39.37 90)
 			(effects
 				(font
@@
 		(dnp no)
 		(property "Reference" "RN307"
-			(at 238.76 34.29 90)
-			(effects
-				(font
-					(size 1.27 1.27)
-				)
-			)
-		)
-		(property "Value" "100K"
-			(at 238.76 39.37 90)
+			(at 238.76 43.942 90)
+			(effects
+				(font
+					(size 1.27 1.27)
+				)
+			)
+		)
+		(property "Value" "4.7K"
+			(at 238.76 41.91 90)
 			(effects
 				(font
@@
 		(dnp no)
 		(property "Reference" "RN306"
-			(at 165.1 86.36 90)
-			(effects
-				(font
-					(size 1.27 1.27)
-				)
-			)
-		)
-		(property "Value" "330R"
-			(at 165.1 91.2876 90)
+			(at 165.1 91.44 90)
+			(effects
+				(font
+					(size 1.27 1.27)
+				)
+			)
+		)
+		(property "Value" "120R"
+			(at 165.1 93.98 90)
 			(effects
 				(font
@@
 		(dnp no)
 		(property "Reference" "RN307"
-			(at 165.1 88.9 90)
-			(effects
-				(font
-					(size 1.27 1.27)
-				)
-			)
-		)
-		(property "Value" "100K"
-			(at 165.1 93.98 90)
-			(effects
-				(font
+			(at 165.1 98.552 90)
+			(effects
+				(font
+					(size 1.27 1.27)
+				)
+			)
+		)
+		(property "Value" "4.7K"
+			(at 165.1 96.52 90)
+			(effects
+				(font
