File: kaybee-plank/kaybee-plank.kicad_sch (KiCad schematic)
At the start: 20 parts, among them J1 Mini-DIN-6, J2 Conn_01x10, J3 Conn_01x10, J4 Mini-DIN-6, J5 USB_A, J7 TYPE-C-31-M-12, J8 Conn_01x02_Pin, SW1 SW_SPDT

Commit message: add szlcsc part numbers
Parts:
- C1, C2, C3: szlcsc_partnum (none) -> C602037
- J1, J4: szlcsc_partnum (none) -> C77848
- J5: szlcsc_partnum (none) -> C456018
- J7: szlcsc_partnum (none) -> C2858270
- J8: szlcsc_partnum (none) -> C2905434
- L1, L2, L4, L5: szlcsc_partnum (none) -> C139190
- R1, R5: szlcsc_partnum (none) -> C27834
- R2, R3: szlcsc_partnum (none) -> C2907315
- SW1: szlcsc_partnum (none) -> C431540
Changed lines of the file:
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@@
+			)
+		)
+		(property "szlcsc_partnum" "C2858270"
+			(at 200.66 93.98 0)
+			(effects
+				(font
+					(size 1.27 1.27)
+				)
+				(hide yes)
 			)
 		)
@@
 			)
 		)
+		(property "szlcsc_partnum" "C77848"
+			(at 171.45 146.05 0)
+			(effects
+				(font
+					(size 1.27 1.27)
+				)
+				(hide yes)
+			)
+		)
 		(pin "1"
 		)
@@
 			)
 		)
+		(property "szlcsc_partnum" "C139190"
+			(at 223.52 83.82 0)
+			(effects
+				(font
+					(size 1.27 1.27)
+				)
+				(hide yes)
+			)
+		)
 		(pin "1"
 		)
@@
 			)
 		)
+		(property "szlcsc_partnum" ""
+			(at 57.15 144.78 0)
+			(effects
+				(font
+					(size 1.27 1.27)
+				)
+				(hide yes)
+			)
+		)
 		(pin "1"
 		)
@@
 			)
 		)
+		(property "szlcsc_partnum" "C139190"
+			(at 118.11 87.63 0)
+			(effects
+				(font
+					(size 1.27 1.27)
+				)
+				(hide yes)
+			)
+		)
 		(pin "1"
 		)
@@
 		)
 		(property "Supplier" "https://item.szlcsc.com/263551.html"
+			(at 152.4 146.05 0)
+			(effects
+				(font
+					(size 1.27 1.27)
+				)
+				(hide yes)
+			)
+		)
+		(property "szlcsc_partnum" "C139190"
 			(at 152.4 146.05 0)
 			(effects
@@
 			)
 		)
+		(property "szlcsc_partnum" "C27834"
+			(at 172.72 88.9 0)
+			(effects
+				(font
+					(size 1.27 1.27)
+				)
+				(hide yes)
+			)
+		)
 		(pin "1"
 		)
@@
 			)
 		)
+		(property "szlcsc_partnum" "C2907315"
+			(at 167.64 36.83 0)
+			(effects
+				(font
+					(size 1.27 1.27)
+				)
+				(hide yes)
+			)
+		)
 		(pin "1"
 		)
@@
 			)
 		)
+		(property "szlcsc_partnum" "C431540"
+			(at 50.8 69.85 0)
+			(effects
+				(font
+					(size 1.27 1.27)
+				)
+				(hide yes)
+			)
+		)
 		(pin "1"
 		)
@@
 		)
 		(property "Supplier" "https://item.szlcsc.com/107087.html"
+			(at 228.6 96.52 0)
+			(effects
+				(font
+					(size 1.27 1.27)
+				)
+				(hide yes)
+			)
+		)
+		(property "szlcsc_partnum" "C27834"
 			(at 228.6 96.52 0)
 			(effects
@@
 			)
 		)
+		(property "szlcsc_partnum" ""
+			(at 34.29 93.98 0)
+			(effects
+				(font
+					(size 1.27 1.27)
+				)
+				(hide yes)
+			)
+		)
 		(pin "1"
 		)
@@
 			)
 		)
+		(property "szlcsc_partnum" "C602037"
+			(at 96.52 41.91 0)
+			(effects
+				(font
+					(size 1.27 1.27)
+				)
+				(hide yes)
+			)
+		)
 		(pin "1"
 		)
@@
 		)
 		(property "Description" "Generic connector, single row, 01x02, script generated"
+			(at 162.56 44.45 0)
+			(effects
+				(font
+					(size 1.27 1.27)
+				)
+				(hide yes)
+			)
+		)
+		(property "szlcsc_partnum" "C2905434"
 			(at 162.56 44.45 0)
 			(effects
@@
 			)
 		)
+		(property "szlcsc_partnum" "C602037"
+			(at 86.36 41.91 0)
+			(effects
+				(font
+					(size 1.27 1.27)
+				)
+				(hide yes)
+			)
+		)
 		(pin "1"
 		)
@@
 			)
 		)
+		(property "szlcsc_partnum" "C456018"
+			(at 105.41 92.71 0)
+			(effects
+				(font
+					(size 1.27 1.27)
+				)
+				(hide yes)
+			)
+		)
 		(pin "3"
 		)
@@
 			)
 		)
+		(property "szlcsc_partnum" "C2907315"
+			(at 49.53 144.78 0)
+			(effects
+				(font
+					(size 1.27 1.27)
+				)
+				(hide yes)
+			)
+		)
 		(pin "1"
 		)
@@
 			)
 		)
+		(property "szlcsc_partnum" "C602037"
+			(at 105.41 41.91 0)
+			(effects
+				(font
+					(size 1.27 1.27)
+				)
+				(hide yes)
+			)
+		)
 		(pin "1"
 		)
@@
 			)
 		)
+		(property "szlcsc_partnum" "C139190"
+			(at 90.17 146.05 0)
+			(effects
+				(font
+					(size 1.27 1.27)
+				)
+				(hide yes)
+			)
+		)
 		(pin "1"
 		)
@@
 		)
 		(property "Description" ""
+			(at 45.72 93.98 0)
+			(effects
+				(font
+					(size 1.27 1.27)
+				)
+				(hide yes)
+			)
+		)
+		(property "szlcsc_partnum" ""
 			(at 45.72 93.98 0)
 			(effects
@@
 			(at 110.49 146.05 0)
 			(effects
+				(font
+					(size 1.27 1.27)
+				)
+				(hide yes)
+			)
+		)
+		(property "szlcsc_partnum" "C77848"
+			(at 110.49 146.05 0)
+			(effects
