File: kaybee-plank/kaybee-plank.kicad_pcb (KiCad board)
At the start: 2 copper layers, 39.5 x 51 mm, 20 parts, among them J1 Mini-DIN-6, J2 Conn_01x10, J3 Conn_01x10, J4 Mini-DIN-6, J5 USB_A, J7 TYPE-C-31-M-12, J8 Conn_01x02_Pin, SW1 SW_SPDT

Commit message: ddr5 hacking board
Other:
- board text added: "DEVICE"
- board text added: "HOST"
- board text added: "PS/2 DEVICE"
- board text added: "PS/2 HOST"
- board text removed: "PS/2 IN"
- board text removed: "PS/2 OUT"
- board text removed: "USB IN"
- board text removed: "USB OUT"
Changed lines of the file:
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@@
 		)
 	)
-	(gr_text "PS/2 IN"
+	(gr_text "PS/2 DEVICE"
 		(at 125.25 112 0)
 		(layer "F.SilkS" knockout)
@@
 		)
 	)
-	(gr_text "USB OUT"
+	(gr_text "HOST"
 		(at 108.5 80.75 180)
 		(layer "F.SilkS" knockout)
@@
 		)
 	)
-	(gr_text "USB IN"
+	(gr_text "DEVICE"
 		(at 125.25 87 180)
 		(layer "F.SilkS" knockout)
@@
 		)
 	)
-	(gr_text "PS/2 OUT"
+	(gr_text "PS/2 HOST"
 		(locked yes)
 		(at 109 112 0)
