File: pcb/6-REV2b/IO-expand-595-mux.kicad_sch (KiCad schematic)
At the start: 75 parts, among them Q300 BC2301T 2.8A, Q301 BC2301T 2.8A, Q302 BC2301T 2.8A, Q303 BC2301T 2.8A, Q304 BC2301T 2.8A, Q305 BC2301T 2.8A, Q306 BC2301T 2.8A, Q307 BC2301T 2.8A, U2 74LVC8T245BQ, U402 CD4067, U404 LMV321, U503 74HCT245BQ, U504 GS324MT/TR, U505 GS324MT/TR, U506 LMV321

Commit message: reorg, but forgot to check changes first :(
Parts:
- gave numbers to parts that had none: 9
Connections:
- net AMUX_S1: now also RN315.3 (R1.1); no longer RN315.4 (R1.1)
- net AMUX_S2: now also RN315.2 (R1.1); no longer RN315.4 (R1.1)
- net AMUX_S3: now also RN315.1 (R1.1); no longer RN315.4 (R1.1)
- net BPIO0: now also RN312.1 (R1.1), RN318.8 (R1.8); no longer RN312.4 (R1.1), RN318.5 (R1.8)
- net BPIO1: now also RN312.2 (R1.1), RN318.7 (R1.8); no longer RN312.4 (R1.1), RN318.5 (R1.8)
- net BPIO2: now also RN312.3 (R1.1), RN318.6 (R1.8); no longer RN312.4 (R1.1), RN318.5 (R1.8)
- net BPIO4: now also RN311.1 (R1.1), RN317.8 (R1.8); no longer RN311.4 (R1.1), RN317.5 (R1.8)
- net BPIO5: now also RN311.2 (R1.1), RN317.7 (R1.8); no longer RN311.4 (R1.1), RN317.5 (R1.8)
- net BPIO6: now also RN311.3 (R1.1), RN317.6 (R1.8); no longer RN311.4 (R1.1), RN317.5 (R1.8)
- net MUX_BPIO1: now also RN401.6 (R1.8); no longer RN401.5 (R1.8)
- net MUX_BPIO2: now also RN401.7 (R1.8); no longer RN401.5 (R1.8)
- net MUX_BPIO3: now also RN401.8 (R1.8); no longer RN401.5 (R1.8)
- net MUX_BPIO5: now also RN400.6 (R1.8); no longer RN400.5 (R1.8)
- net MUX_BPIO6: now also RN400.7 (R1.8); no longer RN400.5 (R1.8)
- net MUX_BPIO7: now also RN400.8 (R1.8); no longer RN400.5 (R1.8)
- net MUX_VREF_VOUT: now also RN402.8 (R1.8); no longer RN402.5 (R1.8)
- net VREG_OUT: now also RN402.7 (R1.8); no longer RN402.5 (R1.8)
- net at U402.20 (I11): now also RN402.1 (R1.1); no longer RN402.4 (R1.1)
- net at U402.21 (I10): now also RN402.2 (R1.1); no longer RN402.4 (R1.1)
- net at U402.3 (I6): now also RN401.3 (R1.1); no longer RN401.4 (R1.1)
- net at U402.4 (I5): now also RN401.2 (R1.1); no longer RN401.4 (R1.1)
- net at U402.5 (I4): now also RN401.1 (R1.1); no longer RN401.4 (R1.1)
- net at U402.7 (I2): now also RN400.3 (R1.1); no longer RN400.4 (R1.1)
- net at U402.8 (I1): now also RN400.2 (R1.1); no longer RN400.4 (R1.1)
- net at U402.9 (I0): now also RN400.1 (R1.1); no longer RN400.4 (R1.1)
- net at U503.14 (B4): now also RN315.8 (R1.8); no longer RN315.5 (R1.8)
- net at U503.15 (B3): now also RN315.7 (R1.8); no longer RN315.5 (R1.8)
- net at U503.16 (B2): now also RN315.6 (R1.8); no longer RN315.5 (R1.8)
- net at Q301.3 (D): now also RN311.8 (R1.8); no longer RN311.5 (R1.8)
- net at Q302.3 (D): now also RN311.7 (R1.8); no longer RN311.5 (R1.8)
- net at Q300.3 (D): now also RN311.6 (R1.8); no longer RN311.5 (R1.8)
- net at Q305.3 (D): now also RN312.8 (R1.8); no longer RN312.5 (R1.8)
- net at Q306.3 (D): now also RN312.7 (R1.8); no longer RN312.5 (R1.8)
- net at Q304.3 (D): now also RN312.6 (R1.8); no longer RN312.5 (R1.8)
- net at D501.2, U504.3 (+): now also RN317.3 (R1.1); no longer RN317.4 (R1.1)
- net at D503.2, U505.10 (+): now also RN318.3 (R1.1); no longer RN318.4 (R1.1)
- net at D502.1, U504.10 (+): now also RN317.2 (R1.1); no longer RN317.4 (R1.1)
- net at D502.2, U504.12 (+): now also RN317.1 (R1.1); no longer RN317.4 (R1.1)
- net at D504.1, U505.5 (+): now also RN318.2 (R1.1); no longer RN318.4 (R1.1)
- net at D504.2, U505.3 (+): now also RN318.1 (R1.1); no longer RN318.4 (R1.1)
