File: pcb/6-REV2b/bpu-current_limiter.kicad_sch (KiCad schematic)
At the start: 45 parts, among them Q401 BCM857, Q402 BC2301T 2.8A, Q601 MMDT3906, Q602 BC2301T 2.8A, U601 GS321A-TR, U602 GSV331-TR, U603 LMV321

Commit message: reorg, but forgot to check changes first :(
Parts:
- gave numbers to parts that had none: 1
