File: pcb/7-REV1/IO-expand-595-mux.kicad_sch (KiCad schematic)
At the start: 42 parts, among them Q2 2N7002KT, U10 LM358_DFN, U11 LM358_DFN, U12 LM358_DFN, U13 LM358_DFN, U2 74LVC8T245BQ, U402 CD4067, U503 74HCT245BQ, U9 LM358_DFN

Commit message: reorg, but forgot to check changes first :(
Parts:
- added C5: 0.1uF, Capacitor_SMD:C_0402_1005Metric, symbol Device:C_Small
- added U17, U18, U5: WS72324Q, Package_DFN_QFN:QFN-16-1EP_3x3mm_P0.5mm_EP1.7x1.7mm, symbol ws72324q:WS72324Q
- added U4: XL9555QF24, Package_DFN_QFN:QFN-24-1EP_4x4mm_P0.5mm_EP2.7x2.7mm, symbol TCA6416RTWT:XL9555QF24
Connections:
- net +3V3: now also C5.2, U4.21 (VCC), U4.23 (ADDR1), U4.24 (ADDR2)
- net DISPLAY_BACKLIGHT: now also U4.13 (P13)
- net DISPLAY_RESET: now also U4.16 (P16)
- net GND: now also C5.1, U4.18 (ADDR0), U4.9 (GND)
- new net CURRENT_EN: U4.12 (P12)
- new net CURRENT_EN_OVERRIDE: U4.10 (P10)
- new net CURRENT_RESET: U4.11 (P11)
- new net I2C_SCL: U4.19 (SCL)
- new net I2C_SDA: U4.20 (SDA)
Other:
- note added: "7-bit I2C Address: 0b0100110 (0x26) 8-bit Write Address: 0b01000010 (0x4C) 8-bit Read Address: 0b01000011 (0x4D)"
