File: pcb/7-rev0a/7-REV0.kicad_pcb (KiCad board)
At the start: 4 copper layers, 60 x 60 mm, 252 parts, among them J201 Conn_01x03, J202 TYPE-C-31-M-12, J301 Conn_01x10, J302 Conn_01x09, Q1 MMBT7002K, Q2 MMBT7002K, Q202 MMBT7002K, Q401 BCM857, Q402 BC2301T 2.8A, Q601 MMDT3906, Q602 BC2301T 2.8A, SW101 TS3425BA 098 2.5H 250gf, SW102 TS3315A 250gf 025, U1 RP2350B, U10 LM358_DFN, U102 W25Q128JVSIQ, U105 MT29F1G01ABAFDWB, U11 LM358_DFN, U12 LM358_DFN, U13 LM358_DFN, U2 74LVC8T245BQ, U3 TLV74311PDBVR, U301 AiP74LVC1T45GC363.TR, U302 AiP74LVC1T45GC363.TR, U303 AiP74LVC1T45GC363.TR, U304 AiP74LVC1T45GC363.TR, U305 AiP74LVC1T45GC363.TR, U306 AiP74LVC1T45GC363.TR, U307 AiP74LVC1T45GC363.TR, U308 AiP74LVC1T45GC363.TR, U4 MCP4725xxx-xCH, U401 ME6211A33PG-N, U402 CD4067, U403 AP2127, U5 MCP4725xxx-xCH, U503 74HCT245BQ, U6 TCA6416RTWT, U601 GS321A-TR, U602 GSV331-TR, U7 TCA6416RTWT, U8 APS6404L-3SQR-ZR, U9 LM358_DFN, Y101 ABM8-272-T3

Commit message: reorg, but forgot to check changes first :(
Parts:
- C10, C11, C201, C202, C401, C402, C404, C407: value 4.7uF -> 10uF/6.3v CL05A106MQ5NUN
- C104, C109, C19, C4, C601: value 2.2uF -> 10uF/6.3v CL05A106MQ5NUN
- C21: value 10uF -> 10uF/6.3v CL05A106MQ5NUN
- R202, R203: value 22R -> 27R
- R6: value 100K -> 10K
Changed lines of the file:
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@@
 			)
 		)
-		(property "Value" "4.7uF"
+		(property "Value" "10uF/6.3v CL05A106MQ5NUN"
 			(at 0 1.17 0)
 			(layer "F.Fab")
@@
 			)
 		)
-		(property "Value" "2.2uF"
+		(property "Value" "10uF/6.3v CL05A106MQ5NUN"
 			(at 0 1.16 0)
 			(layer "F.Fab")
@@
 			)
 		)
-		(property "Value" "22R"
+		(property "Value" "27R"
 			(at 0 1.17 90)
 			(layer "F.Fab")
@@
 			)
 		)
-		(property "Value" "22R"
+		(property "Value" "27R"
 			(at 0 1.17 90)
 			(layer "F.Fab")
@@
 			)
 		)
-		(property "Value" "2.2uF"
+		(property "Value" "10uF/6.3v CL05A106MQ5NUN"
 			(at 0 1.16 90)
 			(layer "F.Fab")
@@
 			)
 		)
-		(property "Value" "4.7uF"
+		(property "Value" "10uF/6.3v CL05A106MQ5NUN"
 			(at 0 1.16 90)
 			(layer "F.Fab")
@@
 			)
 		)
-		(property "Value" "4.7uF"
+		(property "Value" "10uF/6.3v CL05A106MQ5NUN"
 			(at 0 1.16 90)
 			(layer "F.Fab")
@@
 			)
 		)
-		(property "Value" "4.7uF"
+		(property "Value" "10uF/6.3v CL05A106MQ5NUN"
 			(at 0 1.16 90)
 			(layer "F.Fab")
@@
 			)
 		)
-		(property "Value" "2.2uF"
+		(property "Value" "10uF/6.3v CL05A106MQ5NUN"
 			(at 0 1.17 90)
 			(layer "F.Fab")
@@
 			)
 		)
-		(property "Value" "4.7uF"
+		(property "Value" "10uF/6.3v CL05A106MQ5NUN"
 			(at 0 1.16 0)
 			(layer "F.Fab")
@@
 			)
 		)
-		(property "Value" "4.7uF"
+		(property "Value" "10uF/6.3v CL05A106MQ5NUN"
 			(at 0 1.16 90)
 			(layer "F.Fab")
@@
 			)
 		)
-		(property "Value" "4.7uF"
+		(property "Value" "10uF/6.3v CL05A106MQ5NUN"
 			(at 0 1.16 90)
 			(layer "F.Fab")
@@
 			)
 		)
-		(property "Value" "10uF"
+		(property "Value" "10uF/6.3v CL05A106MQ5NUN"
 			(at 0 1.16 0)
 			(layer "F.Fab")
@@
 			)
 		)
-		(property "Value" "4.7uF"
+		(property "Value" "10uF/6.3v CL05A106MQ5NUN"
 			(at 0 1.16 90)
 			(layer "F.Fab")
@@
 			)
 		)
-		(property "Value" "100K"
+		(property "Value" "10K"
 			(at 0 1.17 90)
 			(layer "F.Fab")
@@
 		(sheetname "bpu-iobufffer")
 		(sheetfile "bpu-iobufffer.kicad_sch")
-		(attr smd)
+		(attr smd exclude_from_bom dnp)
 		(fp_line
 			(start 0.7 -0.6)
@@
 			)
 		)
-		(property "Value" "2.2uF"
+		(property "Value" "10uF/6.3v CL05A106MQ5NUN"
 			(at 0 1.16 0)
 			(layer "F.Fab")
@@
 		(sheetname "bpu-iobufffer")
 		(sheetfile "bpu-iobufffer.kicad_sch")
-		(attr smd)
+		(attr smd exclude_from_bom dnp)
 		(fp_line
 			(start 0.7 -0.6)
@@
 		(sheetname "bpu-iobufffer")
 		(sheetfile "bpu-iobufffer.kicad_sch")
-		(attr smd)
+		(attr smd exclude_from_bom dnp)
 		(fp_line
 			(start 0.7 -0.6)
@@
 		(sheetname "bpu-iobufffer")
 		(sheetfile "bpu-iobufffer.kicad_sch")
-		(attr smd)
+		(attr smd exclude_from_bom dnp)
 		(fp_line
 			(start 0.7 -0.6)
@@
 		(sheetname "bpu-iobufffer")
 		(sheetfile "bpu-iobufffer.kicad_sch")
-		(attr smd)
+		(attr smd exclude_from_bom dnp)
 		(fp_line
 			(start 0.7 -0.6)
@@
 			)
 		)
-		(property "Value" "2.2uF"
+		(property "Value" "10uF/6.3v CL05A106MQ5NUN"
 			(at 0 1.16 90)
 			(layer "F.Fab")
@@
 		(sheetname "bpu-iobufffer")
 		(sheetfile "bpu-iobufffer.kicad_sch")
-		(attr smd)
+		(attr smd exclude_from_bom dnp)
 		(fp_line
 			(start 0.7 -0.6)
@@
 		(sheetname "bpu-iobufffer")
 		(sheetfile "bpu-iobufffer.kicad_sch")
-		(attr smd)
+		(attr smd exclude_from_bom dnp)
 		(fp_line
 			(start 0.7 -0.6)
@@
 		(sheetname "bpu-iobufffer")
 		(sheetfile "bpu-iobufffer.kicad_sch")
-		(attr smd)
+		(attr smd exclude_from_bom dnp)
 		(fp_line
 			(start 0.7 -0.6)
@@
 		(sheetname "bpu-iobufffer")
 		(sheetfile "bpu-iobufffer.kicad_sch")
-		(attr smd)
+		(attr smd exclude_from_bom dnp)
 		(fp_line
 			(start 0.7 -0.6)
