File: pcb/7-rev0a/bpu-iobufffer.kicad_sch (KiCad schematic)
At the start: 44 parts, among them J301 Conn_01x10, J302 Conn_01x09, U301 AiP74LVC1T45GC363.TR, U302 AiP74LVC1T45GC363.TR, U303 AiP74LVC1T45GC363.TR, U304 AiP74LVC1T45GC363.TR, U305 AiP74LVC1T45GC363.TR, U306 AiP74LVC1T45GC363.TR, U307 AiP74LVC1T45GC363.TR, U308 AiP74LVC1T45GC363.TR

Commit message: reorg, but forgot to check changes first :(
Parts:
- D10, D11, D12, D13, D14, D15, D16, D17, D18: now not fitted; now left out of the parts list
Changed lines of the file:
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@@
 		(unit 1)
 		(exclude_from_sim no)
-		(in_bom yes)
-		(on_board yes)
-		(dnp no)
+		(in_bom no)
+		(on_board yes)
+		(dnp yes)
 		(property "Reference" "D17"
 			(at 116.84 182.88 0)
@@
 		(unit 1)
 		(exclude_from_sim no)
-		(in_bom yes)
-		(on_board yes)
-		(dnp no)
+		(in_bom no)
+		(on_board yes)
+		(dnp yes)
 		(property "Reference" "D15"
 			(at 101.6 182.88 0)
@@
 		(unit 1)
 		(exclude_from_sim no)
-		(in_bom yes)
-		(on_board yes)
-		(dnp no)
+		(in_bom no)
+		(on_board yes)
+		(dnp yes)
 		(property "Reference" "D16"
 			(at 109.22 182.88 0)
@@
 		(unit 1)
 		(exclude_from_sim no)
-		(in_bom yes)
-		(on_board yes)
-		(dnp no)
+		(in_bom no)
+		(on_board yes)
+		(dnp yes)
 		(property "Reference" "D18"
 			(at 85.09 182.88 0)
@@
 		(unit 1)
 		(exclude_from_sim no)
-		(in_bom yes)
-		(on_board yes)
-		(dnp no)
+		(in_bom no)
+		(on_board yes)
+		(dnp yes)
 		(property "Reference" "D10"
 			(at 147.32 182.88 0)
@@
 		(unit 1)
 		(exclude_from_sim no)
-		(in_bom yes)
-		(on_board yes)
-		(dnp no)
+		(in_bom no)
+		(on_board yes)
+		(dnp yes)
 		(property "Reference" "D12"
 			(at 124.46 182.88 0)
@@
 		(unit 1)
 		(exclude_from_sim no)
-		(in_bom yes)
-		(on_board yes)
-		(dnp no)
+		(in_bom no)
+		(on_board yes)
+		(dnp yes)
 		(property "Reference" "D13"
 			(at 132.08 182.88 0)
@@
 		(unit 1)
 		(exclude_from_sim no)
-		(in_bom yes)
-		(on_board yes)
-		(dnp no)
+		(in_bom no)
+		(on_board yes)
+		(dnp yes)
 		(property "Reference" "D11"
 			(at 139.7 182.88 0)
@@
 		(unit 1)
 		(exclude_from_sim no)
-		(in_bom yes)
-		(on_board yes)
-		(dnp no)
+		(in_bom no)
+		(on_board yes)
+		(dnp yes)
 		(property "Reference" "D14"
 			(at 93.98 182.88 0)
